Commit message: roboclaw integration

File: src/cr_hardware/description/ros2_control/cuberover.ros2_control.xacro (robot description, xacro)
@@ -1,9 +1,10 @@
 <?xml version="1.0"?>
 <robot xmlns:xacro="http://www.ros.org/wiki/xacro">
-  <xacro:macro name="cuberover_ros2_control" params="name prefix use_mock_hardware">
+  <xacro:macro name="cuberover_ros2_control" params="name prefix use_mock_hardware debug">
     <ros2_control name="${name}" type="system">
       <xacro:unless value="${use_mock_hardware}">
         <hardware>
-          <plugin>cr_hardware/DifferentialDriveHardware</plugin>
+          <plugin>cr_hardware/DifferentialDrive</plugin>
+          <param name="debug">${debug}</param>
           <!-- <param name="example_param_hw_start_duration_sec">0</param>
           <param name="example_param_hw_stop_duration_sec">3.0</param> -->

File: src/cr_hardware/description/urdf/cuberover.urdf.xacro (robot description, xacro)
@@ -4,4 +4,5 @@
   <xacro:arg name="prefix" default="" />
   <xacro:arg name="use_mock_hardware" default="false" />
+  <xacro:arg name="debug" default="false" />
   <xacro:include filename="$(find ros2_control_demo_description)/diffbot/urdf/diffbot_description.urdf.xacro" />
   <!-- Import Rviz colors -->
@@ -11,4 +12,7 @@
   <xacro:diffbot prefix="$(arg prefix)" />
   <xacro:cuberover_ros2_control
-    name="DiffBot" prefix="$(arg prefix)" use_mock_hardware="$(arg use_mock_hardware)"/>
+    name="CuberoverDiffDrive"
+    prefix="$(arg prefix)"
+    use_mock_hardware="$(arg use_mock_hardware)"
+    debug="$(arg debug)" />
 </robot>

Commit message: bno055 module

File: src/cr_hardware/description/ros2_control/cuberover.ros2_control.xacro (robot description, xacro)
@@ -1,5 +1,8 @@
 <?xml version="1.0"?>
 <robot xmlns:xacro="http://www.ros.org/wiki/xacro">
-  <xacro:macro name="cuberover_ros2_control" params="name prefix use_mock_hardware debug">
+  <xacro:macro name="cuberover_ros2_control" params="name prefix
+    use_mock_hardware
+    debug
+    serial_port">
     <ros2_control name="${name}" type="system">
       <xacro:unless value="${use_mock_hardware}">
@@ -7,4 +10,5 @@
           <plugin>cr_hardware/DifferentialDrive</plugin>
           <param name="debug">${debug}</param>
+          <param name="serial_port">${serial_port}</param>
           <!-- <param name="example_param_hw_start_duration_sec">0</param>
           <param name="example_param_hw_stop_duration_sec">3.0</param> -->

File: src/cr_hardware/description/urdf/cuberover.urdf.xacro (robot description, xacro)
@@ -5,7 +5,8 @@
   <xacro:arg name="use_mock_hardware" default="false" />
   <xacro:arg name="debug" default="false" />
-  <xacro:include filename="$(find ros2_control_demo_description)/diffbot/urdf/diffbot_description.urdf.xacro" />
+  <xacro:arg name="serial_port" default="/dev/ttyACM0" />
+  <xacro:include filename="$(find cr_hardware)/urdf/diffbot_description.urdf.xacro" />
   <!-- Import Rviz colors -->
-  <xacro:include filename="$(find ros2_control_demo_description)/diffbot/urdf/diffbot.materials.xacro" />
+  <xacro:include filename="$(find cr_hardware)/urdf/diffbot.materials.xacro" />
   <!-- Import cuberover ros2_control description -->
   <xacro:include filename="$(find cr_hardware)/ros2_control/cuberover.ros2_control.xacro" />
@@ -15,4 +16,6 @@
     prefix="$(arg prefix)"
     use_mock_hardware="$(arg use_mock_hardware)"
-    debug="$(arg debug)" />
+    debug="$(arg debug)"
+    serial_port="$(arg serial_port)"
+  />
 </robot>
